File: KiCad/OpenCoil_Driver/OpenCoil_Driver.kicad_pcb (KiCad board)
At the start: 2 copper layers, 0 parts

Commit message: layout experiments
Parts:
- added REF**: PowerPAK_SO-8_Dual, Package_SO:PowerPAK_SO-8_Dual, F.Cu at (203.5, 74.5)
- added REF**: D_SOD-323, Diode_SMD:D_SOD-323, F.Cu at (162.2, 89.2)
- added REF**: SOT-23-6, Package_TO_SOT_SMD:SOT-23-6, F.Cu at (155.8, 96.0)
- added REF**: DFN-8-1EP_3x3mm_P0.65mm_EP1.7x2.05mm, Package_DFN_QFN:DFN-8-1EP_3x3mm_P0.65mm_EP1.7x2.05mm, F.Cu at (157.8, 82.0)
- added REF**: DFN-8-1EP_3x3mm_P0.65mm_EP1.7x2.05mm, Package_DFN_QFN:DFN-8-1EP_3x3mm_P0.65mm_EP1.7x2.05mm, F.Cu at (237.5, 77.1)
- added REF**: Relay_SPDT_Schrack-RT1-FormC_RM3.5mm, Relay_THT:Relay_SPDT_Schrack-RT1-FormC_RM3.5mm, F.Cu at (96.9, 51.2)
- added REF**: D_SOD-323, Diode_SMD:D_SOD-323, F.Cu at (158.2, 89.2)
- added REF**: SOT-23-6, Package_TO_SOT_SMD:SOT-23-6, F.Cu at (163.8, 96.2)
- added REF**: PowerPAK_SO-8_Dual, Package_SO:PowerPAK_SO-8_Dual, F.Cu at (220.0, 74.5)
- added REF**: RJ45_Amphenol_54602-x08_Horizontal, Connector_RJ:RJ45_Amphenol_54602-x08_Horizontal, F.Cu at (164.3, 71.1)
- added REF**: RJ45_Amphenol_54602-x08_Horizontal, Connector_RJ:RJ45_Amphenol_54602-x08_Horizontal, F.Cu at (148.3, 71.1)
- added REF**: D_SOD-323, Diode_SMD:D_SOD-323, F.Cu at (154.2, 89.2)
- added REF**: C_0603_1608Metric, Capacitor_SMD:C_0603_1608Metric, F.Cu at (165.5, 91.8)
- added REF**: TSSOP-8_3x3mm_P0.65mm, Package_SO:TSSOP-8_3x3mm_P0.65mm, F.Cu at (106.5, 102.8)
- added REF**: D_SOD-323, Diode_SMD:D_SOD-323, F.Cu at (166.2, 89.2)
- added REF**: RJ45_Amphenol_54602-x08_Horizontal, Connector_RJ:RJ45_Amphenol_54602-x08_Horizontal, F.Cu at (180.3, 71.1)
- added REF**: MountingHole_3.2mm_M3, MountingHole:MountingHole_3.2mm_M3, F.Cu at (125.0, 81.0)
- added REF**: TSSOP-8_3x3mm_P0.65mm, Package_SO:TSSOP-8_3x3mm_P0.65mm, F.Cu at (206.2, 82.0)
- added REF**: Relay_SPDT_Schrack-RT1-FormC_RM3.5mm, Relay_THT:Relay_SPDT_Schrack-RT1-FormC_RM3.5mm, F.Cu at (83.2, 51.2)
- added REF**: Allegro_CB_PFF, Sensor_Current:Allegro_CB_PFF, F.Cu at (123.6, 47.6)
- added REF**: PowerPAK_SO-8_Dual, Package_SO:PowerPAK_SO-8_Dual, F.Cu at (214.5, 74.5)
- added REF**: TerminalBlock_Phoenix_MKDS-1,5-2_1x02_P5.00mm_Horizontal, TerminalBlock_Phoenix:TerminalBlock_Phoenix_MKDS-1,5-2_1x02_P5.00mm_Horizontal, F.Cu at (131.5, 66.7)
- added REF**: C_0805_2012Metric, Capacitor_SMD:C_0805_2012Metric, F.Cu at (165.5, 85.2)
- added REF**: TSSOP-16_4.4x5mm_P0.65mm, Package_SO:TSSOP-16_4.4x5mm_P0.65mm, F.Cu at (176.5, 108.0)
- added REF**: C_0603_1608Metric, Capacitor_SMD:C_0603_1608Metric, F.Cu at (161.5, 91.8)
- added REF**: MountingHole_3.2mm_M3, MountingHole:MountingHole_3.2mm_M3, F.Cu at (180.0, 136.0)
- added REF**: C_0805_2012Metric, Capacitor_SMD:C_0805_2012Metric, F.Cu at (161.5, 85.2)
- added REF**: R_0603_1608Metric, Resistor_SMD:R_0603_1608Metric, F.Cu at (152.5, 89.2)
- added REF**: TSSOP-8_3x3mm_P0.65mm, Package_SO:TSSOP-8_3x3mm_P0.65mm, F.Cu at (217.2, 82.0)
- added REF**: R_Axial_Power_L20.0mm_W6.4mm_P25.40mm, Resistor_THT:R_Axial_Power_L20.0mm_W6.4mm_P25.40mm, F.Cu at (81.8, 19.0)
- added REF**: DFN-8-1EP_3x3mm_P0.65mm_EP1.7x2.05mm, Package_DFN_QFN:DFN-8-1EP_3x3mm_P0.65mm_EP1.7x2.05mm, F.Cu at (153.8, 82.0)
- added REF**: PowerPAK_SO-8_Dual, Package_SO:PowerPAK_SO-8_Dual, F.Cu at (209.0, 74.5)
- added REF**: DFN-8-1EP_3x3mm_P0.65mm_EP1.7x2.05mm, Package_DFN_QFN:DFN-8-1EP_3x3mm_P0.65mm_EP1.7x2.05mm, F.Cu at (241.5, 77.1)
- added REF**: C_0805_2012Metric, Capacitor_SMD:C_0805_2012Metric, F.Cu at (157.5, 85.2)
- added REF**: MountingHole_3.2mm_M3, MountingHole:MountingHole_3.2mm_M3, F.Cu at (180.0, 81.0)
- added REF**: R_0603_1608Metric, Resistor_SMD:R_0603_1608Metric, F.Cu at (156.5, 89.2)
- added REF**: MountingHole_3.2mm_M3, MountingHole:MountingHole_3.2mm_M3, F.Cu at (125.0, 136.0)
- added REF**: C_0603_1608Metric, Capacitor_SMD:C_0603_1608Metric, F.Cu at (153.5, 91.8)
- added REF**: R_0603_1608Metric, Resistor_SMD:R_0603_1608Metric, F.Cu at (160.5, 89.2)
- added REF**: TSSOP-24_4.4x7.8mm_P0.65mm, Package_SO:TSSOP-24_4.4x7.8mm_P0.65mm, F.Cu at (176.5, 118.0)
- added REF**: C_0805_2012Metric, Capacitor_SMD:C_0805_2012Metric, F.Cu at (153.5, 85.2)
- added REF**: DFN-8-1EP_3x3mm_P0.65mm_EP1.7x2.05mm, Package_DFN_QFN:DFN-8-1EP_3x3mm_P0.65mm_EP1.7x2.05mm, F.Cu at (165.8, 82.0)
- added REF**: DFN-8-1EP_3x3mm_P0.65mm_EP1.7x2.05mm, Package_DFN_QFN:DFN-8-1EP_3x3mm_P0.65mm_EP1.7x2.05mm, F.Cu at (233.5, 77.1)
- added REF**: C_0603_1608Metric, Capacitor_SMD:C_0603_1608Metric, F.Cu at (157.5, 91.8)
- added REF**: DFN-8-1EP_3x3mm_P0.65mm_EP1.7x2.05mm, Package_DFN_QFN:DFN-8-1EP_3x3mm_P0.65mm_EP1.7x2.05mm, F.Cu at (161.8, 82.0)
- added REF**: R_0603_1608Metric, Resistor_SMD:R_0603_1608Metric, F.Cu at (164.5, 89.2)
- added U3: ICE40UP5K-SG48ITR, Package_DFN_QFN:QFN-48-1EP_7x7mm_P0.5mm_EP5.6x5.6mm, F.Cu at (152.5, 111.0)
- added U4: W25Q32JVSS, Package_SO:SOIC-8_5.23x5.23mm_P1.27mm, F.Cu at (138.8, 111.2)
Routing:
- net (no net): track 0.00 -> 70.3 mm, vias 0 -> 2
Other:
- board outline added: 65 x 80 mm
