File: KiCad/OpenCoil_Driver/GateDriver.kicad_sch (KiCad schematic)
At the start: 15 parts, among them U5 2EDN7534BXTSA1, U7 DMC3025LDV, U8 DMC3025LDV

Commit message: schematic structure plan
Connections:
- net INA renamed ~{INA}
- net INB renamed ~{INB}
Changed lines of the file:
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@@
     (stroke (width 0) (type default))
   )
-  (hierarchical_label "INB" (shape input) (at 86.36 95.25 180) (fields_autoplaced)
+  (hierarchical_label "~{INB}" (shape input) (at 86.36 95.25 180) (fields_autoplaced)
     (effects (font (size 1.27 1.27)) (justify right))
   )
@@
     (effects (font (size 1.27 1.27)) (justify left))
   )
-  (hierarchical_label "INA" (shape input) (at 86.36 92.71 180) (fields_autoplaced)
+  (hierarchical_label "~{INA}" (shape input) (at 86.36 92.71 180) (fields_autoplaced)
     (effects (font (size 1.27 1.27)) (justify right))
   )
