File: KiCad/OpenCoil_Driver/OpenCoil_Driver.kicad_sch (KiCad schematic)
At the start: 0 parts

Commit message: Renamed KiCad project
Other:
- title: ProjectTemplate -> OpenCoil_Driver
Changed lines of the file:
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@@
   (paper "A4")
   (title_block
-    (title "ProjectTemplate")
+    (title "OpenCoil_Driver")
     (date "2023-09-16")
     (rev "0")
@@
     (comment 1 "sjsimmo123@gmail.com")
     (comment 2 "Samuel Simmons")
-    (comment 4 "Template Project for KiCad")
+    (comment 4 "Driver PCB for OpenCoil FPGA based tesla coil project")
   )
   (sheet_instances

Commit message: started drafting schematic
Parts:
- added C? (x6): ?, symbol Device:C
- added C?: 10u, symbol Device:C
- added C?: 100n, symbol Device:C
- added D?: D, symbol Device:D
- added J?: POWER INPUT, symbol Connector_Generic:Conn_01x02
- added J?: CT, symbol Connector_Generic:Conn_01x02
- added J?: GDTs, symbol Connector_Generic:Conn_01x04
- added J?: Vmeasure, symbol Connector_Generic:Conn_01x04
- added J?: Tmeasure, symbol Connector_Generic:Conn_01x02
- added R?: 100R, symbol Device:R_US
- added R? (x6): 10k, symbol Device:R_US
- added U?: W25Q32JVSS, Package_SO:SOIC-8_5.23x5.23mm_P1.27mm, symbol Memory_Flash:W25Q32JVSS
- added U? (x4): ICE40UP5K-SG48ITR, Package_DFN_QFN:QFN-48-1EP_7x7mm_P0.5mm_EP5.6x5.6mm, symbol FPGA_Lattice:ICE40UP5K-SG48ITR
- added U?: ADC1173, symbol Analog_ADC:ADC1173
Connections:
- new net: C?.1, C?.1, R?.2, U?.29 (VCCPLL)
- new net: R?.1, U?.3 (IO2)
- new net: R?.1, U?.7 (IO3)
- new net +1V2: R?.1, U?.30 (VCC), U?.5 (VCC)
- new net +2V5: C?.1, D?.1 (K), U?.24 (VPP_2V5)
- new net +3V3: C?.1, D?.2 (A), R?.1, R?.1, R?.2, R?.2, R?.2, R?.2, U?.1 (VCCIO_2), U?.22 (SPI_VCCIO1), U?.33 (VCCIO_0), U?.8 (VCC)
- new net CDONE: R?.2, U?.7 (CDONE)
- new net FLASH_MISO: U?.17 (IOB_33b_SPI_SI), U?.2 (DO(IO1))
- new net FLASH_MOSI: U?.14 (IOB_32a_SPI_SO), U?.5 (DI(IO0))
- new net FLASH_SCK: R?.1, U?.15 (IOB_34a_SPI_SCK), U?.6 (CLK)
- new net FLASH_~{CS}: R?.1, U?.1 (~{CS}), U?.16 (IOB_35b_SPI_SS)
- new net GND: C?.2, C?.2, C?.2, C?.2, U?.4 (GND), U?.49 (GND)
- new net ~{CRESET}: R?.2, U?.8 (~{CRESET})
Other:
- note added: "+24VDC GND"
- note added: "A+ A- B+ B-"
- note added: "Prog Interface"
- note added: "Tsnk+ Tsnk-"
- note added: "Vbus+ Vbus- Vout+ Vout-"
- note added: "https://hackaday.io/project/163794/gallery#40c5674bfafc014f09bd6637c6192bac"
- note added: "min 104161bytes or 833288bits"

Commit message: draft CT input stage
Parts:
- removed C? (x2): ?, symbol Device:C
- removed J?: POWER INPUT, symbol Connector_Generic:Conn_01x02
- removed J?: GDTs, symbol Connector_Generic:Conn_01x04
- removed J?: Vmeasure, symbol Connector_Generic:Conn_01x04
- removed J?: Tmeasure, symbol Connector_Generic:Conn_01x02
- removed U?: ADC1173, symbol Analog_ADC:ADC1173
- added C? (x2): 10u, symbol Device:C
- added C? (x8): C, symbol Device:C
- added C? (x6): 100n, symbol Device:C
- added C? (x4): ?, symbol Device:C
- added D1, D2, D3, D4: D_Schottky, symbol Device:D_Schottky
- added D? (x4): B5819WS, symbol Device:D
- added J11: Conn_02x04_Odd_Even, symbol Connector_Generic:Conn_02x04_Odd_Even
- added L1: L, symbol Device:L
- added Q? (x4): NMOS, symbol Simulation_SPICE:NMOS
- added Q? (x4): PMOS, symbol Simulation_SPICE:PMOS
- added R1, R2, R3, R4: R_US, symbol Device:R_US
- added R? (x2): R, symbol Device:R_US
- added R? (x4): 1k, symbol Device:R_US
- added U1: Comparator, symbol Simulation_SPICE:OPAMP
- added U2: ADC08060, symbol Analog_ADC:ADC08060
- C?: value ? -> 100n
Connections:
- net +3V3: now also C?.1, C?.1, C?.1, C?.1, C?.1, C?.1, C?.1, J11.1 (Pin_1), L1.2, U1.4 (V+), U2.18 (DVDD)
- net CDONE: now also J11.3 (Pin_3)
- net FLASH_MISO: now also J11.8 (Pin_8)
- net FLASH_MOSI: now also J11.2 (Pin_2)
- net FLASH_SCK: now also J11.4 (Pin_4)
- net FLASH_~{CS}: now also J11.6 (Pin_6)
- net GND: now also C?.2, C?.2, C?.1, C?.1, C?.1, C?.1, C?.1, C?.1, C?.2, C?.2, C?.2, C?.2, C?.2, C?.2, D2.2 (A), D4.2 (A), J11.7 (Pin_7), Q?.3 (S), Q?.3 (S), Q?.3 (S), Q?.3 (S), R3.2, U1.5 (V-), U2.10 (VRB), U2.11 (AGND), U2.17 (DGND), U2.2 (AGND), U2.23 (PWR_DWN), U2.5 (AGND), U2.7 (VIN_GND), U2.8 (DGND), U2.9 (VRB)
- net ~{CRESET}: now also J11.5 (Pin_5)
- net at J?.1 (Pin_1): now also D1.2 (A), D2.1 (K), R2.1
- net at J?.2 (Pin_2): now also D3.2 (A), D4.1 (K), R1.1
- new net: C?.2, Q?.1 (D), Q?.1 (D), R?.1 (x2)
- new net: C?.2, R?.2 (x2)
- new net: C?.2, C?.2, L1.1, U2.1 (AVDD), U2.12 (AVDD), U2.4 (AVDD)
- new net: C?.1, R4.2, U2.6 (AIN)
- new net: Q?.1 (D), Q?.1 (D) (x2)
- new net: C?.2, Q?.2 (G) (x4)
- new net: C?.1, D?.2 (A), Q?.2 (G), R?.2 (x4)
- new net: C?.1, C?.1 (x2)
- new net: R1.2, U1.2 (-)
- new net: R2.2, U1.1 (+)
- new net +24V: C?.2, C?.2, C?.2, C?.2, D?.1 (K), D?.1 (K), D?.1 (K), D?.1 (K), Q?.3 (S), Q?.3 (S), Q?.3 (S), Q?.3 (S), R?.1, R?.1, R?.1, R?.1
- new net I_ADC0: U2.13 (D0), U2.14 (D1), U2.15 (D2), U2.16 (D3), U2.19 (D4), U2.20 (D5), U2.21 (D6), U2.22 (D7)
- new net I_ADC_CLK: U2.24 (CLK)
- new net I_MAG: D1.1 (K), D3.1 (K), R3.1, R4.1
- new net I_ZCS: U1.3
Other:
- note added: "+24V"
- note added: "+5V"
- note added: "Auxiliary"
- note added: "Bridge"
- note added: "CT+"
- note added: "CT-"
- note added: "FAN"
- note added: "Flash Programming Interface"
- note added: "GDT1+"
- note added: "GDT1-"
- note added: "GDT2+"
- note added: "GDT2-"
- note added: "GND"
- note added: "GPIO1"
- note added: "GPIO2"
- note added: "Isense"
- note added: "LED_B"
- note added: "LED_G"
- note added: "LED_R"
- note added: "Power Input"
- note added: "RL1"
- note added: "RL2"
- note added: "Soft Start"
- note added: "TLV3501?"
- note added: "TODO: UVLO?"
- note added: "Tsense+"
- note added: "Tsense-"
- note added: "Vsense+"
- note added: "Vsense-"
- note removed: "+24VDC GND"
- note removed: "A+ A- B+ B-"
- note removed: "Prog Interface"
- note removed: "Tsnk+ Tsnk-"
- note removed: "Vbus+ Vbus- Vout+ Vout-"
- moved on the sheet: C?, D?, J?, R?, U?, U?A, U?B, U?C, U?D

Commit message: add DMC3025
Parts:
- removed Q? (x4): NMOS, symbol Simulation_SPICE:NMOS
- removed Q? (x4): PMOS, symbol Simulation_SPICE:PMOS
- added U5, U6, U7, U8: DMC3025LDV, Package_SON:Diodes_PowerDI3333-8_UXC_3.3x3.3mm_P0.65mm, symbol KiCadLibrary:DMC3025LDV
- gave numbers to parts that had none: 22
- renumbered J11 to J2
Connections:
- net +24V: now also U5.3 (S), U6.3 (S), U7.3 (S), U8.3 (S)
- net GND: now also U5.1 (S), U6.1 (S), U7.1 (S), U8.1 (S)
- net at C23.2, R16.1: now also U5.5 (D), U5.7 (D)
- net at C24.2, R17.1: now also U7.5 (D), U7.7 (D)
- net at C18.2: now also U8.2 (G)
- net at C16.1, D7.2 (A), R13.2: now also U6.4 (G)
- net at C16.2: now also U6.2 (G)
- net at C17.1, D8.2 (A), R14.2: now also U7.4 (G)
- net at C18.1, D9.2 (A), R15.2: now also U8.4 (G)
- net at C15.1, D6.2 (A), R12.2: now also U5.4 (G)
- net at C15.2: now also U5.2 (G)
- net at C17.2: now also U7.2 (G)
- new net: U8.5 (D), U8.7 (D)
- new net: U6.5 (D), U6.7 (D)

Commit message: move to hierarchical design
Parts:
- removed C15, C16, C17, C18, C?: 100n, symbol Device:C
- removed C19, C20, C21, C22, C23, C24, C25, C26: C, symbol Device:C
- removed C? (x2): ?, symbol Device:C
- removed C?: 10u, symbol Device:C
- removed D6, D7, D8, D9: B5819WS, symbol Device:D
- removed D?: D, symbol Device:D
- removed R12, R13, R14, R15: 1k, symbol Device:R_US
- removed R16, R17: R, symbol Device:R_US
- removed R?: 100R, symbol Device:R_US
- removed U5, U6, U7, U8: DMC3025LDV, Package_SON:Diodes_PowerDI3333-8_UXC_3.3x3.3mm_P0.65mm, symbol KiCadLibrary:DMC3025LDV
- removed U?: ICE40UP5K-SG48ITR, Package_DFN_QFN:QFN-48-1EP_7x7mm_P0.5mm_EP5.6x5.6mm, symbol FPGA_Lattice:ICE40UP5K-SG48ITR
- added C?: 100n, symbol Device:C
- added C?: 10u, symbol Device:C
- added J?: RJ45_Shielded, symbol Connector:RJ45_Shielded
- added R?: 100R, symbol Device:R_US
- added U?: ICE40UP5K-SG48ITR, Package_DFN_QFN:QFN-48-1EP_7x7mm_P0.5mm_EP5.6x5.6mm, symbol FPGA_Lattice:ICE40UP5K-SG48ITR
Connections:
- net +1V2: now also R?.1, U?.30 (VCC), U?.5 (VCC)
- net +2V5: now also U?.24 (VPP_2V5)
- net GND: now also C?.2, C?.2, J?.SH, U?.49 (GND)
- new net: C?.1, C?.1, R?.2, U?.29 (VCCPLL)
- new net GDT_1A: J?.4
- new net GDT_1B: J?.5
- new net GDT_2A: J?.3
- new net GDT_2B: J?.6
Other:
- added sheet Gate Driver 1 (GateDriver.kicad_sch)
- added sheet Gate Driver 2 (GateDriver.kicad_sch)
- added sheet Regulators (Regulators.kicad_sch)
- note added: "min 104161bytes or 833288bits - more for RISC-V"
- note removed: "TODO: UVLO?"
- note removed: "min 104161bytes or 833288bits"
- moved on the sheet: C?, R?, U?B

Commit message: add connectors, general cleanup
Parts:
- removed J?: RJ45_Shielded, symbol Connector:RJ45_Shielded
- added J? (x3): RJ45_Shielded, symbol Connector:RJ45_Shielded
- added J?: Screw_Terminal_01x02, symbol Connector:Screw_Terminal_01x02
Connections:
- net GDT_1A: now also J?.4
- net GDT_1B: now also J?.5
- net GDT_2A: now also J?.3
- net GDT_2B: now also J?.6
- net GND: now also J?.2 (Pin_2), J?.6, J?.6, J?.SH, J?.SH, J?.SH
- new net +24V: J?.1 (Pin_1), J?.8, J?.8
- new net +5V: J?.7
- new net CT_A: J?.8
- new net CT_B: J?.7
- new net FAN: J?.7
- new net GPIO_1: J?.2
- new net GPIO_2: J?.1
- new net Isense: J?.3
- new net LED_B: J?.3
- new net LED_G: J?.4
- new net LED_R: J?.5
- new net RL_1: J?.2
- new net RL_2: J?.1
- new net Tsense+: J?.2
- new net Tsense-: J?.1
- new net Vsense+: J?.5
- new net Vsense-: J?.4
Other:
- note added: "Connectors"
- note added: "FPGA and Flash Storage"
- note added: "Sheets"
- note removed: "+24V"
- note removed: "+5V"
- note removed: "CT+"
- note removed: "CT-"
- note removed: "FAN"
- note removed: "GDT1+"
- note removed: "GDT1-"
- note removed: "GDT2+"
- note removed: "GDT2-"
- note removed: "GND"
- note removed: "GPIO1"
- note removed: "GPIO2"
- note removed: "Isense"
- note removed: "LED_B"
- note removed: "LED_G"
- note removed: "LED_R"
- note removed: "RL1"
- note removed: "RL2"
- note removed: "Tsense+"
- note removed: "Tsense-"
- note removed: "Vsense+"
- note removed: "Vsense-"
- moved on the sheet: C?, J2, R?, U?, U?A, U?B, U?C, U?D

Commit message: schematic structure plan
Parts:
- removed C?: 100n, symbol Device:C
- removed C?: 10u, symbol Device:C
- removed R? (x2): 10k, symbol Device:R_US
- removed R?: 100R, symbol Device:R_US
- removed U?: ICE40UP5K-SG48ITR, Package_DFN_QFN:QFN-48-1EP_7x7mm_P0.5mm_EP5.6x5.6mm, symbol FPGA_Lattice:ICE40UP5K-SG48ITR
- added R? (x2): 10k, symbol Device:R_US
Connections:
- net +3V3: now also R?.1, R?.1
- net CDONE: now also R?.2
- net ~{CRESET}: now also R?.2
- net FLASH_IO2: now reaches R?.1, U?.3 (IO2)
- net FLASH_IO3: now reaches R?.1, U?.7 (IO3)
- net FAN renamed ~{FAN}
- net LED_B renamed ~{LED_B}
- net LED_G renamed ~{LED_G}
- net LED_R renamed ~{LED_R}
- net RL_1 renamed ~{RL_1}
- net RL_2 renamed ~{RL_2}
Other:
- added sheet ADC (ADC.kicad_sch)
- added sheet Analog Inputs (AnalogInputs.kicad_sch)
- added sheet CT Input (CTInput.kicad_sch)
- sheet Gate Driver 1 ports: added ~{INA}, ~{INB}; removed INA, INB
- sheet Gate Driver 2 ports: added ~{INA}, ~{INB}; removed INA, INB
- note added: "FPGA IO"
- note added: "Submodules"
- note added: "TODO: REF?"
- note added: "TODO: TLV3501?"
- note added: "TODO: https://hackaday.io/project/163794/gallery#40c5674bfafc014f09bd6637c6192bac"
- note added: "TODO: min 104161bytes or 833288bits - more for RISC-V"
- note removed: "FPGA and Flash Storage"
- note removed: "Sheets"
- note removed: "TLV3501?"
- note removed: "https://hackaday.io/project/163794/gallery#40c5674bfafc014f09bd6637c6192bac"
- note removed: "min 104161bytes or 833288bits - more for RISC-V"
- moved on the sheet: C?, J2, J?, R?, U?, U?A, U?B, U?C
