File: KiCad/OpenCoil_Driver/Regulators.kicad_sch (KiCad schematic)
At the start: 3 parts

Commit message: schematic structure plan
Parts:
- added C?: 100n, symbol Device:C
- added C?: 10u, symbol Device:C
- added R?: 100R, symbol Device:R_US
- added U?: ICE40UP5K-SG48ITR, Package_DFN_QFN:QFN-48-1EP_7x7mm_P0.5mm_EP5.6x5.6mm, symbol FPGA_Lattice:ICE40UP5K-SG48ITR
Connections:
- net +1V2: now also R?.1, U?.30 (VCC), U?.5 (VCC)
- net +2V5: now also U?.24 (VPP_2V5)
- net GND: now also C?.2, C?.2, U?.49 (GND)
- new net: C?.1, C?.1, R?.2, U?.29 (VCCPLL)
Other:
- note added: "TODO: - UVLO? - Fuse? - +5V - +3V3 - +2V5 - +1V2"
- note removed: "TODO: UVLO?"
